Commit message: updated model

File: cyton_gamma_1500.urdf (robot description, URDF)
Before this commit: robot cyton_gamma_1500, 12 links, 11 joints
Links:
- link elbow_pitch: geometry collision box size=0.0549 0.1557 0.076; visual mesh filename=package://cyton_gamma_1500_description/meshes/elbow_pitch.d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
- link elbow_yaw: geometry collision box size=0.0535 0.1160 0.0402; visual mesh filename=package://cyton_gamma_1500_description/meshes/elbow_yaw.dae
- link shoulder_pitch: geometry collision box size=0.0709 0.19363 0.083; visual mesh filename=package://cyton_gamma_1500_description/meshes/shoulder_pitc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
- link shoulder_roll: geometry collision box size=0.09829 0.18143 0.08392; visual mesh filename=package://cyton_gamma_1500_description/meshes/shoulder_roll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
- link shoulder_yaw: geometry collision box size=0.0717 0.1846 0.0756; visual mesh filename=package://cyton_gamma_1500_description/meshes/shoulder_yaw.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
- link wrist_pitch: geometry collision box size=0.026 0.0435 0.05185; visual mesh filename=package://cyton_gamma_1500_description/meshes/wrist_pitch.d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
- link wrist_roll: geometry collision box size=0.0518 0.0723 0.1004; visual mesh filename=package://cyton_gamma_1500_description/meshes/wrist_roll.dae
Joints:
- joint elbow_pitch_joint: origin xyz=0.018 0.0215 0.1158 rpy=0 0 0 -> xyz=0.018 0.0206 0.1158 rpy=0 0 0
- joint elbow_yaw_joint: origin xyz=-0.0185 -0.018 0.0973 rpy=0 0 0 -> xyz=-0.0171 -0.018 0.09746 rpy=0 0 0
- joint gripper_joint: origin xyz=0.008 -0.00305 0.08868 rpy=0 0 0 -> xyz=-0.01331 0.00485 0.077225 rpy=0 0 0
- joint gripper_joint2: origin xyz=-0.008 -0.00305 0.08868 rpy=0 0 0 -> xyz=0.0098 0.00485 0.077225 rpy=0 0 0
- joint shoulder_roll_joint: origin xyz=0 0 0.053 rpy=0 0 0 -> xyz=0 0 0.05315 rpy=0 0 0
- joint virtual_endeffector_joint: origin xyz=0 0 0.090875 rpy=0 0 0 -> xyz=-0.002316 0.0079 0.079425 rpy=0 0 0
- joint wrist_pitch_joint: origin xyz=0.02325 0.018 0.0718 rpy=0 0 0 -> xyz=0.02626 0.018 0.0718 rpy=0 0 0
- joint wrist_roll_joint: origin xyz=-0.02625 0 0.05142 rpy=0 0 0 -> xyz=-0.026255 0 0.051425 rpy=0 0 0

File: cyton_gamma_1500_macros.urdf.xacro (robot description, xacro)
@@ -37,5 +37,5 @@
       <parent link="${prefix}base_link" />
       <child link="${prefix}shoulder_roll" />
-      <origin xyz="0 0 0.053" rpy="0 0 0" />
+      <origin xyz="0 0 0.05315" rpy="0 0 0" />
       <limit lower="-2.618" upper="2.618" effort="100.0" velocity="1.0" />
       <axis xyz="0 0 1" />
@@ -43,5 +43,5 @@
     <link name="${prefix}shoulder_roll">
       <visual>
-        <origin xyz="0 0 0" rpy="0 -1.5708 3.5256"/>
+        <origin xyz="0 0 0" rpy="1.5708 0 0.384"/>
         <geometry>
           <mesh filename="package://cyton_gamma_1500_description/meshes/shoulder_roll.dae"/>
@@ -49,7 +49,7 @@
       </visual>
       <collision>
-        <origin xyz="0.069 0.0055 0.0544"/>
-        <geometry>
-          <box size="0.18143 0.0839 0.0955"/>
+        <origin xyz="0.0 0.069 0.0587"/>
+        <geometry>
+          <box size="0.09829 0.18143 0.08392"/>
         </geometry>
       </collision>
@@ -70,7 +70,7 @@
       </visual>
       <collision>
-        <origin xyz="-0.001 0.064 0.1759"/>
-        <geometry>
-          <box size="0.0709 0.1936 0.08"/>
+        <origin xyz="-0.001 0.064 0.1745"/>
+        <geometry>
+          <box size="0.0709 0.19363 0.083"/>
         </geometry>
       </collision>
@@ -91,7 +91,7 @@
       </visual>
       <collision>
-        <origin xyz="-0.0225 0.039 0.3052"/>
-        <geometry>
-          <box size="0.0717 0.1846 0.0726"/>
+        <origin xyz="-0.0225 0.039 0.3068"/>
+        <geometry>
+          <box size="0.0717 0.1846 0.0756"/>
         </geometry>
       </collision>
@@ -100,5 +100,5 @@
       <parent link="${prefix}shoulder_yaw" />
       <child link="${prefix}elbow_pitch" />
-      <origin xyz="0.018 0.0215 0.1158" rpy="0 0 0" />
+      <origin xyz="0.018 0.0206 0.1158" rpy="0 0 0" />
       <limit lower="-1.8326" upper="1.8326" effort="100.0" velocity="1.0" />
       <axis xyz="1 0 0" />
@@ -112,7 +112,7 @@
       </visual>
       <collision>
-        <origin xyz="0.0346 0.046 0.4214"/>
-        <geometry>
-          <box size="0.0549 0.1556 0.0735"/>
+        <origin xyz="0.0346 0.0461 0.4228"/>
+        <geometry>
+          <box size="0.0549 0.1557 0.076"/>
         </geometry>
       </collision>
@@ -121,5 +121,5 @@
       <parent link="${prefix}elbow_pitch" />
       <child link="${prefix}elbow_yaw" />
-      <origin xyz="-0.0185 -0.018 0.0973" rpy="0 0 0" />
+      <origin xyz="-0.0171 -0.018 0.09746" rpy="0 0 0" />
       <limit lower="-1.8326" upper="1.8326" effort="100.0" velocity="1.0" />
       <axis xyz="0 -1 0" />
@@ -133,7 +133,7 @@
       </visual>
       <collision>
-        <origin xyz="0.0162 0.0211 0.516"/>
-        <geometry>
-          <box size="0.0535 0.1165 0.0402"/>
+        <origin xyz="0.0172 0.0209 0.516"/>
+        <geometry>
+          <box size="0.0535 0.1160 0.0402"/>
         </geometry>
       </collision>
@@ -142,5 +142,5 @@
       <parent link="${prefix}elbow_yaw" />
       <child link="${prefix}wrist_pitch" />
-      <origin xyz="0.02325 0.018 0.0718" rpy="0 0 0" />
+      <origin xyz="0.02626 0.018 0.0718" rpy="0 0 0" />
       <limit lower="-1.8326" upper="1.8326" effort="100.0" velocity="1.0" />
       <axis xyz="1 0 0" />
@@ -154,7 +154,7 @@
       </visual>
       <collision>
-        <origin xyz="0.0248 0.0118 0.5614"/>
-        <geometry>
-          <box size="0.026 0.0435 0.0519"/>
+        <origin xyz="0.0257 0.0118 0.5617"/>
+        <geometry>
+          <box size="0.026 0.0435 0.05185"/>
         </geometry>
       </collision>
@@ -163,5 +163,5 @@
       <parent link="${prefix}wrist_pitch" />
       <child link="${prefix}wrist_roll" />
-      <origin xyz="-0.02625 0 0.05142" rpy="0 0 0" />
+      <origin xyz="-0.026255 0 0.051425" rpy="0 0 0" />
       <limit lower="-2.61799" upper="2.61799" effort="100.0" velocity="1.0" />
       <axis xyz="0 0 1" />
@@ -175,7 +175,7 @@
       </visual>
       <collision>
-        <origin xyz="0.0022 -0.003 0.6042"/>
-        <geometry>
-          <box size="0.0546 0.0745 0.1118"/>
+        <origin xyz="-0.0063 -0.0014 0.6102"/>
+        <geometry>
+          <box size="0.0518 0.0723 0.1004"/>
         </geometry>
       </collision>
@@ -184,5 +184,5 @@
       <parent link="${prefix}wrist_roll" />
       <child link="${prefix}gripper_finger1" />
-      <origin xyz="0.008 -0.00305 0.08868" rpy="0 0 0" />
+      <origin xyz="-0.01331 0.00485 0.077225" rpy="0 0 0" />
       <limit lower="-0.008" upper="0.008" effort="100.0" velocity="1.0" />
       <axis xyz="1 0 0" />
@@ -196,5 +196,5 @@
       </visual>
       <collision>
-        <origin xyz="0.0135 0.0093 0.7365"/>
+        <origin xyz="-0.0167 0.0172 0.7254"/>
         <geometry>
           <box size="0.015 0.0229 0.0475"/>
@@ -205,5 +205,5 @@
       <parent link="${prefix}wrist_roll" />
       <child link="${prefix}gripper_finger2" />
-      <origin xyz="-0.008 -0.00305 0.08868" rpy="0 0 0" />
+      <origin xyz="0.0098 0.00485 0.077225" rpy="0 0 0" />
       <limit lower="-0.008" upper="0.008" effort="100.0" velocity="1.0" />
       <mimic joint="${prefix}gripper_joint" multiplier="-1"/>
@@ -218,5 +218,5 @@
       </visual>
       <collision>
-        <origin xyz="-0.0175 0.0093 0.7365"/>
+        <origin xyz="0.0132 0.0172 0.7254"/>
         <geometry>
           <box size="0.015 0.0229 0.0475"/>
@@ -224,9 +224,9 @@
       </collision>
     </link>
-    <xacro:if value="${virtual_ee}"> <!-- virtual point end-effector -->
+    <xacro:if value="${virtual_ee}"> <!-- virtual end-effector -->
       <joint name="${prefix}virtual_endeffector_joint" type="fixed">
         <parent link="${prefix}wrist_roll" />
         <child link="${prefix}virtual_endeffector" />
-        <origin xyz="0 0 0.090875" rpy="0 0 0" />
+        <origin xyz="-0.002316 0.0079 0.079425" rpy="0 0 0" />
       </joint>
       <link name="${prefix}virtual_endeffector">

Commit message: Fixed one axis and updated models (removed emission lighting)

File: cyton_gamma_1500.urdf (robot description, URDF)
Before this commit: robot cyton_gamma_1500, 12 links, 11 joints
Joints:
- joint wrist_pitch_joint: axis 1 0 0 -> -1 0 0

File: cyton_gamma_1500_macros.urdf.xacro (robot description, xacro)
@@ -144,5 +144,5 @@
       <origin xyz="0.02626 0.018 0.0718" rpy="0 0 0" />
       <limit lower="-1.8326" upper="1.8326" effort="100.0" velocity="1.0" />
-      <axis xyz="1 0 0" />
+      <axis xyz="-1 0 0" />
     </joint>
     <link name="${prefix}wrist_pitch">

Commit message: updates for gazebo

File: cyton_gamma_1500.urdf (robot description, URDF)
Before this commit: robot cyton_gamma_1500, 12 links, 11 joints
Links:
- link base_link: mass None -> 100.0
- link elbow_pitch: mass None -> 10.0
- link elbow_yaw: mass None -> 10.0
- link gripper_finger1: mass None -> 1.0
- link gripper_finger2: mass None -> 1.0
- link shoulder_pitch: mass None -> 20.0
- link shoulder_roll: mass None -> 50.0
- link shoulder_yaw: mass None -> 10.0
- link wrist_pitch: mass None -> 10.0
- link wrist_roll: mass None -> 10.0
