Commit message: adding in the xacro for the urdf file

File: cyton_gamma_1500_macros.urdf.xacro (robot description, xacro)
@@ -33,4 +33,10 @@
         </geometry>
       </collision>
+      <inertial>
+        <mass value="100.0"/>
+        <origin rpy="0 0 0" xyz="0 0 0"/>
+        <inertia ixx="1.1027" iyy="1.1027" izz="1.1027"
+                  ixy="0" ixz="0" iyz="0"/>
+      </inertial>
     </link>
     <joint name="${prefix}shoulder_roll_joint" type="revolute">
@@ -54,4 +60,10 @@
         </geometry>
       </collision>
+      <inertial>
+        <mass value="50.0"/>
+        <origin rpy="0 0 0" xyz="0 0 0"/>
+        <inertia ixx=".1027" iyy=".1027" izz=".1027"
+                  ixy="0" ixz="0" iyz="0"/>
+      </inertial>
     </link>
     <joint name="${prefix}shoulder_pitch_joint" type="revolute">
@@ -75,4 +87,10 @@
         </geometry>
       </collision>
+      <inertial>
+        <mass value="20.0"/>
+        <origin rpy="0 0 0" xyz="0 0 0"/>
+        <inertia ixx=".0827" iyy=".0827" izz=".0827"
+                  ixy="0" ixz="0" iyz="0"/>
+      </inertial>
     </link>
     <joint name="${prefix}shoulder_yaw_joint" type="revolute">
@@ -96,4 +114,10 @@
         </geometry>
       </collision>
+      <inertial>
+        <mass value="10.0"/>
+        <origin rpy="0 0 0" xyz="0 0 0"/>
+        <inertia ixx=".0627" iyy=".0627" izz=".0627"
+                  ixy="0" ixz="0" iyz="0"/>
+      </inertial>
     </link>
     <joint name="${prefix}elbow_pitch_joint" type="revolute">
@@ -117,4 +141,10 @@
         </geometry>
       </collision>
+      <inertial>
+        <mass value="10.0"/>
+        <origin rpy="0 0 0" xyz="0 0 0"/>
+        <inertia ixx=".0327" iyy=".0327" izz=".0327"
+                  ixy="0" ixz="0" iyz="0"/>
+      </inertial>
     </link>
     <joint name="${prefix}elbow_yaw_joint" type="revolute">
@@ -138,4 +168,10 @@
         </geometry>
       </collision>
+      <inertial>
+        <mass value="10.0"/>
+        <origin rpy="0 0 0" xyz="0 0 0"/>
+        <inertia ixx=".0227" iyy=".0227" izz=".0227"
+                  ixy="0" ixz="0" iyz="0"/>
+      </inertial>
     </link>
     <joint name="${prefix}wrist_pitch_joint" type="revolute">
@@ -159,4 +195,10 @@
         </geometry>
       </collision>
+      <inertial>
+        <mass value="10.0"/>
+        <origin rpy="0 0 0" xyz="0 0 0"/>
+        <inertia ixx=".0127" iyy=".0127" izz=".0127"
+                  ixy="0" ixz="0" iyz="0"/>
+      </inertial>
     </link>
     <joint name="${prefix}wrist_roll_joint" type="revolute">
@@ -180,4 +222,10 @@
         </geometry>
       </collision>
+      <inertial>
+        <mass value="10.0"/>
+        <origin rpy="0 0 0" xyz="0 0 0"/>
+        <inertia ixx=".0027" iyy=".0027" izz=".0027"
+                  ixy="0" ixz="0" iyz="0"/>
+      </inertial>
     </link>
     <joint name="${prefix}gripper_joint" type="prismatic">
@@ -201,4 +249,10 @@
         </geometry>
       </collision>
+      <inertial>
+        <mass value="1.0"/>
+        <origin rpy="0 0 0" xyz="0 0 0"/>
+        <inertia ixx=".0027" iyy=".0027" izz=".0027"
+                  ixy="0" ixz="0" iyz="0"/>
+      </inertial>
     </link>
     <joint name="${prefix}gripper_joint2" type="prismatic">
@@ -223,4 +277,10 @@
         </geometry>
       </collision>
+      <inertial>
+        <mass value="1.0"/>
+        <origin rpy="0 0 0" xyz="0 0 0"/>
+        <inertia ixx=".0027" iyy=".0027" izz=".0027"
+                  ixy="0" ixz="0" iyz="0"/>
+      </inertial>
     </link>
     <xacro:if value="${virtual_ee}"> <!-- virtual end-effector -->
@@ -243,3 +303,12 @@
     </xacro:if>
   </xacro:macro>
+  <gazebo>
+    <plugin name="gazebo_ros_control" filename="libgazebo_ros_control.so"/>
+  </gazebo>
+  <gazebo>
+    <plugin name="joint_state_publisher"
+            filename="libgazebo_ros_joint_state_publisher.so">
+      <jointName>shoulder_roll_joint, shoulder_pitch_joint, shoulder_yaw_joint, elbow_pitch_joint, elbow_yaw_joint, wrist_pitch_joint, wrist_roll_joint, gripper_joint, gripper_joint2</jointName>
+    </plugin>
+  </gazebo>
 </robot>

Commit message: allow prefix in base_footprint link

File: cyton_gamma_1500_macros.urdf.xacro (robot description, xacro)
@@ -2,5 +2,5 @@
 <robot xmlns:xacro="http://www.ros.org/wiki/xacro" name="cyton_gamma_1500">
   <xacro:macro name="base_footprint" params="prefix">
-    <link name="base_footprint">
+    <link name="${prefix}base_footprint">
       <visual>
         <origin xyz="0 0 0" rpy="0 0 0"/>
@@ -14,5 +14,5 @@
     </link>
     <joint name="base_joint" type="fixed">
-      <parent link="base_footprint" />
+      <parent link="${prefix}base_footprint" />
       <child link="${prefix}base_link" />
       <origin xyz="0.0 0.0 0.0" rpy="0 0 0" />
